File: RelayHK4100F/RelayHK4100F.kicad_pcb (KiCad board)
At the start: 2 copper layers, 31.7 x 15.2 mm, 3 parts, among them J1 Conn_01x05, K1 Y14x-1C-xxDS

Commit message: medir cosas
Other:
- board size 31.7 x 15.2 mm -> 31.1 x 14 mm
Changed lines of the file:
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@@
   )
   (gr_circle (center 134.62 86.36) (end 133.35 85.09) (layer "Edge.Cuts") (width 0.1) (fill none))
-  (gr_rect (start 111.76 78.74) (end 143.51 93.98) (layer "Edge.Cuts") (width 0.1) (fill none))
+  (gr_rect (start 111.76 79.375) (end 142.875 93.345) (layer "Edge.Cuts") (width 0.1) (fill none))
   (dimension (type aligned) (layer "Dwgs.User")
     (pts (xy 110.49 78.74) (xy 110.49 93.98))
     (height 2.54)
     (gr_text "15.2400 mm" (at 106.8 86.36 90) (layer "Dwgs.User")
+      (effects (font (size 1 1) (thickness 0.15)))
+    )
+    (format (units 3) (units_format 1) (precision 4))
+    (style (thickness 0.15) (arrow_length 1.27) (text_position_mode 0) (extension_height 0.58642) (extension_offset 0.5) keep_text_aligned)
+  )
+  (dimension (type aligned) (layer "Dwgs.User")
+    (pts (xy 114.3 81.28) (xy 111.76 81.28))
+    (height 3.809999)
+    (gr_text "2.5400 mm" (at 113.03 76.320001) (layer "Dwgs.User")
+      (effects (font (size 1 1) (thickness 0.15)))
+    )
+    (format (units 3) (units_format 1) (precision 4))
+    (style (thickness 0.15) (arrow_length 1.27) (text_position_mode 0) (extension_height 0.58642) (extension_offset 0.5) keep_text_aligned)
+  )
+  (dimension (type aligned) (layer "Dwgs.User")
+    (pts (xy 143.51 79.375) (xy 143.51 93.345))
+    (height -2.54)
+    (gr_text "13.9700 mm" (at 144.9 86.36 90) (layer "Dwgs.User")
+      (effects (font (size 1 1) (thickness 0.15)))
+    )
+    (format (units 3) (units_format 1) (precision 4))
+    (style (thickness 0.15) (arrow_length 1.27) (text_position_mode 0) (extension_height 0.58642) (extension_offset 0.5) keep_text_aligned)
+  )
+  (dimension (type aligned) (layer "Dwgs.User")
+    (pts (xy 117.475 83.82) (xy 119.38 83.82))
+    (height -3.175)
+    (gr_text "1.9050 mm" (at 118.4275 79.495) (layer "Dwgs.User")
+      (effects (font (size 1 1) (thickness 0.15)))
+    )
+    (format (units 3) (units_format 1) (precision 4))
+    (style (thickness 0.15) (arrow_length 1.27) (text_position_mode 0) (extension_height 0.58642) (extension_offset 0.5) keep_text_aligned)
+  )
+  (dimension (type aligned) (layer "Dwgs.User")
+    (pts (xy 142.875 93.98) (xy 112.395 93.98))
+    (height -7.62)
+    (gr_text "30.4800 mm" (at 127.635 100.45) (layer "Dwgs.User")
+      (effects (font (size 1 1) (thickness 0.15)))
+    )
+    (format (units 3) (units_format 1) (precision 4))
+    (style (thickness 0.15) (arrow_length 1.27) (text_position_mode 0) (extension_height 0.58642) (extension_offset 0.5) keep_text_aligned)
+  )
+  (dimension (type aligned) (layer "Dwgs.User")
+    (pts (xy 134.62 86.36) (xy 112.83 86.36))
+    (height -10.16)
+    (gr_text "21.7900 mm" (at 123.725 95.37) (layer "Dwgs.User")
+      (effects (font (size 1 1) (thickness 0.15)))
+    )
+    (format (units 3) (units_format 1) (precision 4))
+    (style (thickness 0.15) (arrow_length 1.27) (text_position_mode 0) (extension_height 0.58642) (extension_offset 0.5) keep_text_aligned)
+  )
+  (dimension (type aligned) (layer "Dwgs.User")
+    (pts (xy 139.72 95.25) (xy 142.875 95.25))
+    (height 3.175)
+    (gr_text "3.1550 mm" (at 141.2975 97.275) (layer "Dwgs.User")
+      (effects (font (size 1 1) (thickness 0.15)))
+    )
+    (format (units 3) (units_format 1) (precision 4))
+    (style (thickness 0.15) (arrow_length 1.27) (text_position_mode 0) (extension_height 0.58642) (extension_offset 0.5) keep_text_aligned)
+  )
+  (dimension (type aligned) (layer "Dwgs.User")
+    (pts (xy 139.7 76.2) (xy 142.24 76.2))
+    (height -2.54)
+    (gr_text "2.5400 mm" (at 140.97 72.51) (layer "Dwgs.User")
+      (effects (font (size 1 1) (thickness 0.15)))
+    )
+    (format (units 3) (units_format 1) (precision 4))
+    (style (thickness 0.15) (arrow_length 1.27) (text_position_mode 0) (extension_height 0.58642) (extension_offset 0.5) keep_text_aligned)
+  )
+  (dimension (type aligned) (layer "Dwgs.User")
+    (pts (xy 132.715 84.455) (xy 117.475 84.455))
+    (height 6.985)
+    (gr_text "15.2400 mm" (at 125.095 76.32) (layer "Dwgs.User")
+      (effects (font (size 1 1) (thickness 0.15)))
+    )
+    (format (units 3) (units_format 1) (precision 4))
+    (style (thickness 0.15) (arrow_length 1.27) (text_position_mode 0) (extension_height 0.58642) (extension_offset 0.5) keep_text_aligned)
+  )
+  (dimension (type aligned) (layer "Dwgs.User")
+    (pts (xy 129.54 83.82) (xy 121.92 83.82))
+    (height 13.97)
+    (gr_text "7.6200 mm" (at 125.73 68.7) (layer "Dwgs.User")
       (effects (font (size 1 1) (thickness 0.15)))
     )
@@
       (effects (font (size 1 1) (thickness 0.15)))
     )
+    (format (units 3) (units_format 1) (precision 4))
+    (style (thickness 0.15) (arrow_length 1.27) (text_position_mode 0) (extension_height 0.58642) (extension_offset 0.5) keep_text_aligned)
+  )
+  (dimension (type aligned) (layer "Dwgs.User")
+    (pts (xy 134.62 86.36) (xy 142.875 86.36))
+    (height 9.525)
+    (gr_text "8.2550 mm" (at 138.7475 94.735) (layer "Dwgs.User")
+      (effects (font (size 1 1) (thickness 0.15)))
+    )
+    (format (units 3) (units_format 1) (precision 4))
+    (style (thickness 0.15) (arrow_length 1.27) (text_position_mode 0) (extension_height 0.58642) (extension_offset 0.5) keep_text_aligned)
+  )
+  (dimension (type aligned) (layer "Dwgs.User")
+    (pts (xy 121.92 83.82) (xy 119.38 83.82))
+    (height 11.43)
+    (gr_text "2.5400 mm" (at 120.65 71.24) (layer "Dwgs.User")
+      (effects (font (size 1 1) (thickness 0.15)))
+    )
